Commit message: finsihed model (i think)

File: src/rob_bot/urdf/rob_bot.xacro (robot description, xacro)
@@ -151,9 +151,69 @@
     </joint>
     <!-- end rear right wheel -->
+    <!-- kinect camera -->
     <link name='camera'>
+        <inertial>
+            <mass value="0.1"/>
+            <origin xyz="0.0 0 0" rpy=" 0 0 0"/>
+            <inertia ixx="1e-6" ixy="0" ixz="0" iyy="1e-6" iyz="0" izz="1e-6"/>
+        </inertial>
+        <collision name='collision'>
+            <origin xyz="0.0 0 0" rpy=" 0 0 0"/>
+            <geometry>
+                <box size="0.073000 0.276000 0.07200"/>
+            </geometry>
+        </collision>
         <visual name='camera_visual'>
+            <origin xyz="0.0 0 0" rpy=" 0 0 0"/>
+            <geometry>
+                <mesh filename="package://rob_bot/meshes/kinect.dae"/>
+            </geometry>
+        </visual>
+    </link>
+    <joint type="fixed" name="camera_link">
+        <origin xyz="0.2 0 0.1" rpy="0 0 0"/>
+        <child link="camera"/>
+        <parent link="chassis"/>
+    </joint>
+    <joint name="camera_depth_joint" type="fixed">
+        <origin xyz="0 0 0" rpy="-1.5707 0 -1.5707"/>
+        <parent link="camera"/>
+        <child link="camera_rgbd_frame"/>
+    </joint>
+    <link name="camera_rgbd_frame"/>
+    <!-- end kinect -->
+    <!-- begin scanner mount -->
+    <!-- raise scanner up 10cm -->
+    <link name='scanner_mount'>
+        <inertial>
+            <mass value="0.1"/>
+            <origin xyz="0.0 0 0" rpy=" 0 0 0"/>
+            <inertia ixx="0.1" ixy="0" ixz="0" iyy="0.1" iyz="0" izz="0.1" />
+        </inertial>
+        <collision name='scanner_mount_collision'>
+            <origin xyz="0 0 0" rpy=" 0 0 0"/>
+            <geometry>
+                <box size=".1 .1 .1"/>
+            </geometry>
+        </collision>
+        <visual name='scanner_mount_visual'>
+            <origin xyz="0 0 0" rpy=" 0 0 0"/>
+            <geometry>
+                <box size=".1 .1 .1"/>
+            </geometry>
+        </visual>
+    </link>
+    <joint type='fixed' name='scanner_mount_to_chasis'>
+        <origin xyz='0 0 0.1' rpy='0 0 0'/>
+        <child link='scanner_mount'/>
+        <parent link='chassis'/>
+    </joint>
+    <!-- end scanner mount -->
+    <!-- begin laser scanner -->
+    <link name='hokuyo'>
+        <visual name='hokuyo_visual'>
             <origin xyz="0 0 0" rpy="0 0 0"/>
             <geometry>
-                <box size='0.05 0.05 0.05'/>
+                <mesh filename="package://rob_bot/meshes/hokuyo.dae"/>
             </geometry>
         </visual>
@@ -166,36 +226,13 @@
             <origin xyz="0 0 0" rpy="0 0 0"/>
             <geometry>
-                <box size='0.05 0.05 0.05'/>
-            </geometry>
-        </collision>
-    </link>
-    <joint type="fixed" name="camera_joint">
-        <origin xyz="0.2 0 0" rpy="0 0 0"/>
-        <child link="camera"/>
-        <parent link="chassis"/>
-    </joint>
-    <link name='hokuyo'>
-        <visual name='hokuyo_visual'>
-            <origin xyz="0 0 0" rpy="0 0 0"/>
-            <geometry>
-                <mesh filename="package://rob_bot/meshes/hokuyo.dae"/>
-            </geometry>
-        </visual>
-        <inertial>
-            <mass value="0.1"/>
-            <origin xyz="0.0 0 0" rpy="0 0 0"/>
-            <inertia ixx="1e-6" ixy="0" ixz="0" iyy="1e-6" iyz="0" izz="1e-6"/>
-        </inertial>
-        <collision name='collision'>
-            <origin xyz="0 0 0" rpy="0 0 0"/>
-            <geometry>
                 <box size='0.1 0.1 0.1'/>
             </geometry>
         </collision>
     </link>
-    <joint type="fixed" name="hokuyo_joint">
-        <origin xyz="0.15 0 0.1" rpy="0 0 0"/>
+    <joint type="fixed" name="hokuyo_to_scanner_mount">
+        <origin xyz="0 0 0.1" rpy="0 0 0"/>
         <child link="hokuyo"/>
-        <parent link="chassis"/>
-    </joint>
+        <parent link="scanner_mount"/>
+    </joint>
+    <!-- end laser scanner -->
 </robot>

Commit message: trying in workspace

File: src/rob_bot/urdf/rob_bot.xacro (robot description, xacro)
@@ -176,6 +176,6 @@
         <parent link="chassis"/>
     </joint>
-    <joint name="camera_depth_joint" type="fixed">
-        <origin xyz="0 0 0" rpy="-1.5707 0 -1.5707"/>
+    <joint name="camera_rgbd_joint" type="fixed">
+        <origin xyz="0 0 0" rpy="-${pi/2} 0 -${pi/2}"/>
         <parent link="camera"/>
         <child link="camera_rgbd_frame"/>
